File: MPPT.sch (KiCad schematic (older format))
At the start: 122 parts, among them J1 Solar Array, J2 Battery, J3 Car Power, J4 CAN_In, J5 CAN_Out, Q1 NMOS, Q2 NMOS, SW1 RESET, SW2 CAN Address, U1 PQMC3-D12-S9-S, U2 Nucleo_L432KC, U3 UCC37321, U4 INA210, U5 ADM3055E, U6 INA210, U7 CDSOT23-T24CAN

Commit message: Major MPPT Board overhaul. Schematic advanced to Rev 3.2. Layout advanced to Rev 1.3. README and documentation updated. Parts list synchronized, standardized, and referenced.
Parts:
- removed LED4: Battery Full?, LEDs:LED_0805_HandSoldering, symbol LED_ALT
- removed R15: 330R, Resistors_SMD:R_0805_HandSoldering, symbol R_Small
- removed SW2: CAN Address, Buttons_Switches_THT:SW_DIP_x4_W7.62mm_Slide_LowProfile, symbol SW_DIP_x04
- added F1: Fuse, MPPT-PrimaryPCB:05200101Z_Fuze_Holder_5x20_PCB_Mount, symbol Device:Fuse
- added H1: Top Left Mounting Hole, MountingHole:MountingHole_3.2mm_M3, symbol Mechanical:MountingHole
- added H2: Top Right Mounting Hole, MountingHole:MountingHole_3.2mm_M3, symbol Mechanical:MountingHole
- added H3: Bottom Left Mounting Hole, MountingHole:MountingHole_3.2mm_M3, symbol Mechanical:MountingHole
- added H4: Bottom Right Mounting Hole, MountingHole:MountingHole_3.2mm_M3, symbol Mechanical:MountingHole
- added HS1: Schottky Diode Heatsink, Heatsink:Heatsink_Fischer_SK129-STS_42x25mm_2xDrill2.5mm, symbol Mechanical:Heatsink
- added HS2: Snubber Heatsink, Heatsink:Heatsink_Fischer_SK129-STS_42x25mm_2xDrill2.5mm, symbol Mechanical:Heatsink
- added HS3: MOSFET Heatsink, Heatsink:Heatsink_Fischer_SK129-STS_42x25mm_2xDrill2.5mm, symbol Mechanical:Heatsink
- added LED10: BPS Full (Blue), LED_SMD:LED_0805_2012Metric, symbol Device:LED_ALT
- added LED5: Error (Amber), LED_SMD:LED_0805_2012Metric, symbol Device:LED_ALT
- added R11, R6: 330, Resistor_SMD:R_0805_2012Metric, symbol Device:R_Small
- added SW2: SW_DIP_x02, MPPT-PrimaryPCB:ADF02ST04_DIP_Switch_2_POS, symbol Switch:SW_DIP_x02
- added U6, U7: MAX40075AUT+, Package_TO_SOT_SMD:SOT-23-6, symbol Array:MAX400_option2-Amplifier_Current
- C1: renamed from C6; value 0.1u -> 0.1uF; footprint Capacitors_SMD:C_0805_HandSoldering -> Capacitor_SMD:C_0805_2012Metric; symbol C_Small -> Device:C_Small
- C10: renamed from C2; footprint UTSVT_Passive:CP_Radial_D31mm_P9mm -> Capacitor_THT:CP_Radial_D30.0mm_P10.00mm_SnapIn; symbol CP1 -> Device:CP1
- C11: renamed from C17; footprint Capacitors_SMD:C_0805_HandSoldering -> Capacitor_SMD:C_0805_2012Metric; symbol C_Small -> Device:C_Small
- C12: renamed from C21; footprint Capacitors_SMD:C_0805_HandSoldering -> Capacitor_SMD:C_0805_2012Metric; symbol C_Small -> Device:C_Small
- C13: renamed from C18; footprint Capacitors_SMD:C_0805_HandSoldering -> Capacitor_SMD:C_0805_2012Metric; symbol C_Small -> Device:C_Small
- C14: renamed from C22; footprint Capacitors_SMD:C_0805_HandSoldering -> Capacitor_SMD:C_0805_2012Metric; symbol C_Small -> Device:C_Small
- C15: renamed from C19; footprint Capacitors_SMD:C_0805_HandSoldering -> Capacitor_SMD:C_0805_2012Metric; symbol C_Small -> Device:C_Small
- C16: renamed from C20; footprint Capacitors_SMD:C_0805_HandSoldering -> Capacitor_SMD:C_0805_2012Metric; symbol C_Small -> Device:C_Small
- C17: renamed from C13; value 10u -> 10uF; footprint Capacitors_SMD:C_0805 -> Capacitor_SMD:C_0805_2012Metric; symbol C_Small -> Device:C_Small
- C18: renamed from C14; value 0.1u -> 0.1uF; footprint Capacitors_SMD:C_0805 -> Capacitor_SMD:C_0805_2012Metric; symbol C_Small -> Device:C_Small
- C19: renamed from C15; value 0.1u -> 0.1uF; footprint Capacitors_SMD:C_0805 -> Capacitor_SMD:C_0805_2012Metric; symbol C_Small -> Device:C_Small
- C2: renamed from C7; value 1u -> 1uF; footprint Capacitors_THT:CP_Radial_D10.0mm_P5.00mm -> Capacitor_SMD:C_0805_2012Metric; symbol C_Small -> Device:C_Small
- C20: renamed from C16; value 0.01u -> 0.01uF; footprint Capacitors_SMD:C_0805 -> Capacitor_SMD:C_0805_2012Metric; symbol C_Small -> Device:C_Small
- C21: renamed from C10; value 0.22u -> 0.22uF; footprint Capacitors_SMD:C_0805_HandSoldering -> Capacitor_SMD:C_0805_2012Metric; symbol C_Small -> Device:C_Small
- C22: renamed from C9; value 10u -> 10uF; footprint Capacitors_SMD:C_0805_HandSoldering -> Capacitor_SMD:C_0805_2012Metric; symbol C_Small -> Device:C_Small
- C23: renamed from C12; value 0.01u -> 0.01uF; footprint Capacitors_SMD:C_0805_HandSoldering -> Capacitor_SMD:C_0805_2012Metric; symbol C_Small -> Device:C_Small
- C24: renamed from C11; value 0.1u -> 0.1uF; footprint Capacitors_SMD:C_0805_HandSoldering -> Capacitor_SMD:C_0805_2012Metric; symbol C_Small -> Device:C_Small
- C3: renamed from C8; value 0.1u -> 0.1uF; footprint Capacitors_SMD:C_0805_HandSoldering -> Capacitor_SMD:C_0805_2012Metric; symbol C_Small -> Device:C_Small
- C4: renamed from C24; value 100u -> 100uF; footprint Capacitors_SMD:CP_Elec_6.3x7.7 -> Capacitor_SMD:C_1210_3225Metric; symbol CP1_Small -> Device:CP1_Small
- C5: renamed from C4; value 47u -> 47uF; footprint Capacitors_SMD:CP_Elec_6.3x5.3 -> Capacitor_SMD:C_1210_3225Metric; symbol CP1_Small -> Device:CP1_Small
- C6: renamed from C23; value 10u -> 10uF; footprint Capacitors_SMD:C_0805_HandSoldering -> Capacitor_SMD:C_0805_2012Metric; symbol C_Small -> Device:C_Small
- C7: renamed from C5; value 100u -> 100uF; footprint Capacitors_SMD:CP_Elec_6.3x7.7 -> Capacitor_SMD:C_1210_3225Metric; symbol CP1_Small -> Device:CP1_Small
- C8: renamed from C1; footprint UTSVT_Passive:CP_Radial_D31mm_P9mm -> Capacitor_THT:CP_Radial_D30.0mm_P10.00mm_SnapIn; symbol CP1 -> Device:CP1
- C9: renamed from C3; footprint MPPT_Custom:C_Rect_L26.5mm_W17.0mm_P22.50mm_MKS4 -> Capacitor_THT:C_Rect_L16.5mm_W7.0mm_P15.00mm_MKT; symbol CP1 -> Device:C
- D1: renamed from D9; value 4V Zener -> 3.9V Zener; footprint Diodes_SMD:D_SOD-123F -> Diode_SMD:D_SOD-123F; symbol D_Zener_Small_ALT -> Device:D_Zener_Small_ALT
- D10: renamed from D14; footprint Diodes_SMD:D_SOD-123 -> Diode_SMD:D_SOD-123F; symbol D_ALT -> Device:D_ALT
- D11: renamed from D5; value 4V Zener -> 3.9V Zener; footprint Diodes_SMD:D_SOD-123F -> Diode_SMD:D_SOD-123F; symbol D_Zener_ALT -> Device:D_Zener_ALT
- D12: renamed from D6; footprint Diodes_SMD:D_SOD-123 -> Diode_SMD:D_SOD-123F; symbol D_ALT -> Device:D_ALT
- D13: renamed from D7; value 4V Zener -> 3.9V Zener; footprint Diodes_SMD:D_SOD-123F -> Diode_SMD:D_SOD-123F; symbol D_Zener_ALT -> Device:D_Zener_ALT
- D14: renamed from D8; footprint Diodes_SMD:D_SOD-123 -> Diode_SMD:D_SOD-123F; symbol D_ALT -> Device:D_ALT
- D2: renamed from D10; footprint Diodes_SMD:D_SOD-123 -> Diode_SMD:D_SOD-123F; symbol D_Small_ALT -> Device:D_Small_ALT
- D3: renamed from D4; value 18V Zener -> 16.3V Zener; footprint Diodes_SMD:D_SMA_Handsoldering -> Diode_SMD:D_SOD-123F; symbol D_Zener_ALT -> Device:D_Zener_ALT
- D4: renamed from D1; footprint TO_SOT_Packages_THT:TO-220-2_Vertical -> Package_TO_SOT_THT:TO-220-2_Vertical; symbol D_Schottky -> Device:D_Schottky
- D5: renamed from D2; footprint TO_SOT_Packages_THT:TO-220-2_Vertical -> Package_TO_SOT_THT:TO-220-2_Vertical; symbol D_Schottky -> Device:D_Schottky
- D6: renamed from D3; footprint TO_SOT_Packages_THT:TO-220-2_Vertical -> Package_TO_SOT_THT:TO-220-2_Vertical; symbol D_Schottky -> Device:D_Schottky
- D7: renamed from D11; value 4V Zener -> 3.9V Zener; footprint Diodes_SMD:D_SOD-123F -> Diode_SMD:D_SOD-123F; symbol D_Zener_ALT -> Device:D_Zener_ALT
- D8: renamed from D12; footprint Diodes_SMD:D_SOD-123 -> Diode_SMD:D_SOD-123F; symbol D_ALT -> Device:D_ALT
- D9: renamed from D13; value 4V Zener -> 3.9V Zener; footprint Diodes_SMD:D_SOD-123F -> Diode_SMD:D_SOD-123F; symbol D_Zener_ALT -> Device:D_Zener_ALT
- F2: renamed from F1; footprint UTSVT_Passive:LittelFuse_OMNIBLOK_520Series_PCB -> MPPT-PrimaryPCB:05200101Z_Fuze_Holder_5x20_PCB_Mount; symbol Fuse -> Device:Fuse
- J1: renamed from J3; footprint UTSVT_Connectors:Molex_MicroFit3.0_1x2xP3.00mm_PolarizingPeg_Vertical -> Connector_Molex:Molex_Micro-Fit_3.0_43650-0215_1x02_P3.00mm_Vertical; symbol CarPowerConnector -> Array:PWR_Connector_43650-0215
- J2: renamed from J1; footprint UTSVT_Connectors:PhoenixContact_PowerCombicon5_GF_3x7.62mm -> MPPT-PrimaryPCB:PhoenixContact_PowerCombicon5_GF_2x7.62mm; symbol SolarArrayConnector -> Array:PWR_Connector_1720796
- J3: renamed from J2; footprint UTSVT_Connectors:PhoenixContact_PowerCombicon5_GF_2x7.62mm -> MPPT-PrimaryPCB:PhoenixContact_PowerCombicon5_GF_2x7.62mm; symbol BatteryConnector -> Array:PWR_Connector_1720796
- J4, J5: footprint UTSVT_Connectors:Molex_MicroFit3.0_1x4xP3.00mm_PolarizingPeg_Vertical -> Connector_Molex:Molex_Micro-Fit_3.0_43650-0415_1x04_P3.00mm_Vertical; symbol CANConnector -> Array:CAN_Connector_43650-0427
- JP1: footprint Pin_Headers:Pin_Header_Straight_1x02_Pitch2.54mm -> Connector_PinHeader_2.54mm:PinHeader_1x02_P2.54mm_Vertical; symbol Jumper_NO_Small -> Device:Jumper_NO_Small
- L1: renamed from L4; value 4.7u -> 4.7uH; footprint Inductors_SMD:L_0805_HandSoldering -> Inductor_SMD:L_0805_2012Metric; symbol L_Small -> Device:L_Small
- L2: renamed from L1; footprint Inductors_THT:L_Toroid_Vertical_L46.0mm_W19.1mm_P21.80mm_Bourns_5700 -> MPPT-PrimaryPCB:L_Toroid_Vertical_L46.0mm_W19.1mm_P21.80mm_Bourns_5700; symbol L_Core_Ferrite -> Device:L_Core_Ferrite
- L3: renamed from L2; value 2k -> 1.8kH; footprint Inductors_SMD:L_0805_HandSoldering -> Inductor_SMD:L_0805_2012Metric; symbol Ferrite_Bead_Small -> Device:Ferrite_Bead_Small
- L4: renamed from L3; value 2k -> 1.8kH; footprint Inductors_SMD:L_0805_HandSoldering -> Inductor_SMD:L_0805_2012Metric; symbol Ferrite_Bead_Small -> Device:Ferrite_Bead_Small
- LED1: value Array Live? -> Array Live (Green); footprint LEDs:LED_0805_HandSoldering -> LED_SMD:LED_0805_2012Metric; symbol LED_ALT -> Device:LED_ALT
- LED2: value Battery Live? -> Battery Live (Green); footprint LEDs:LED_0805_HandSoldering -> LED_SMD:LED_0805_2012Metric; symbol LED_ALT -> Device:LED_ALT
- LED3: value Car Power Live? -> Car Power Live (Green); footprint LEDs:LED_0805_HandSoldering -> LED_SMD:LED_0805_2012Metric; symbol LED_ALT -> Device:LED_ALT
- LED4: renamed from LED7; value Iso 9V Live? -> Device 9V Live (Green); footprint LEDs:LED_0805_HandSoldering -> LED_SMD:LED_0805_2012Metric; symbol LED_ALT -> Device:LED_ALT
- LED6: renamed from LED5; value Tracking? -> Tracking (Blue); footprint LEDs:LED_0805_HandSoldering -> LED_SMD:LED_0805_2012Metric; symbol LED_ALT -> Device:LED_ALT
- LED7: renamed from LED6; value PWM -> PWM (Blue); footprint LEDs:LED_0805_HandSoldering -> LED_SMD:LED_0805_2012Metric; symbol LED_ALT -> Device:LED_ALT
- LED8: value CAN_Tx -> CAN_Tx (Blue); footprint LEDs:LED_0805_HandSoldering -> LED_SMD:LED_0805_2012Metric; symbol LED_ALT -> Device:LED_ALT
- LED9: value CAN_Rx -> CAN_Rx (Blue); footprint LEDs:LED_0805_HandSoldering -> LED_SMD:LED_0805_2012Metric; symbol LED_ALT -> Device:LED_ALT
- Q1, Q2: footprint TO_SOT_Packages_THT:TO-247_TO-3P_Vertical -> Package_TO_SOT_THT:TO-247-3_Vertical; symbol Q_NMOS_GDS -> Device:Q_NMOS_GDS
- R1: renamed from R7; value 1R5 -> 1.5; footprint Resistors_SMD:R_1206_HandSoldering -> Resistor_SMD:R_0805_2012Metric; symbol R -> Device:R
- R10: renamed from R22; value 330R -> 330; footprint Resistors_SMD:R_0805_HandSoldering -> Resistor_SMD:R_0805_2012Metric; symbol R_Small -> Device:R_Small
- R12: renamed from R2; footprint Resistors_SMD:R_1206_HandSoldering -> Resistor_SMD:R_0805_2012Metric; symbol R -> Device:R
- R13: renamed from R1; footprint Resistors_THT:R_Axial_Power_L20.0mm_W6.4mm_P22.40mm -> Package_TO_SOT_THT:TO-220-2_Vertical; symbol R -> Device:R
- R14: renamed from R8; footprint Resistors_SMD:R_2512_HandSoldering -> Resistor_SMD:R_1206_3216Metric; symbol R_Small -> Device:R_Small
- R15: renamed from R18; footprint Resistors_SMD:R_0805_HandSoldering -> Resistor_SMD:R_0805_2012Metric; symbol R_Small -> Device:R_Small
- R16: renamed from R11; footprint Resistors_SMD:R_2512_HandSoldering -> Resistor_SMD:R_1206_3216Metric; symbol R_Small -> Device:R_Small
- R17: renamed from R19; footprint Resistors_SMD:R_0805_HandSoldering -> Resistor_SMD:R_0805_2012Metric; symbol R_Small -> Device:R_Small
- R18: renamed from R3; footprint Resistors_SMD:R_1206_HandSoldering -> Resistor_SMD:R_0805_2012Metric; symbol R -> Device:R
- R19: renamed from R5; footprint Resistors_SMD:R_1206_HandSoldering -> Resistor_SMD:R_0805_2012Metric; symbol R -> Device:R
- R2: renamed from R12; value 40K -> 15k; footprint Resistors_SMD:R_1206_HandSoldering -> Resistor_SMD:R_1206_3216Metric; symbol R_Small -> Device:R_Small
- R20: renamed from R23; footprint Resistors_SMD:R_0805_HandSoldering -> Resistor_SMD:R_0805_2012Metric; symbol R_Small -> Device:R
- R21: renamed from R4; footprint Resistors_SMD:R_1206_HandSoldering -> Resistor_SMD:R_0805_2012Metric; symbol R -> Device:R
- R22: renamed from R6; footprint Resistors_SMD:R_1206_HandSoldering -> Resistor_SMD:R_0805_2012Metric; symbol R -> Device:R
- R23: renamed from R24; footprint Resistors_SMD:R_0805_HandSoldering -> Resistor_SMD:R_0805_2012Metric; symbol R_Small -> Device:R
- R24: renamed from R25; footprint Resistors_SMD:R_0805_HandSoldering -> Resistor_SMD:R_0805_2012Metric; symbol R -> Device:R
- R25: renamed from R10; footprint Resistors_SMD:R_0805_HandSoldering -> Resistor_SMD:R_0805_2012Metric; symbol R -> Device:R
- R26: renamed from R9; footprint Resistors_SMD:R_0805_HandSoldering -> Resistor_SMD:R_0805_2012Metric; symbol R -> Device:R
- R3: renamed from R13; value 40K -> 27k; footprint Resistors_SMD:R_1206_HandSoldering -> Resistor_SMD:R_1206_3216Metric; symbol R_Small -> Device:R_Small
- R4: renamed from R14; value 2K -> 1.5k; footprint Resistors_SMD:R_0805_HandSoldering -> Resistor_SMD:R_0805_2012Metric; symbol R_Small -> Device:R_Small
- R5: renamed from R20; value 1K -> 1.1k; footprint Resistors_SMD:R_0805_HandSoldering -> Resistor_SMD:R_0805_2012Metric; symbol R_Small -> Device:R_Small
- R7: renamed from R16; value 330R -> 330; footprint Resistors_SMD:R_0805_HandSoldering -> Resistor_SMD:R_0805_2012Metric; symbol R_Small -> Device:R_Small
- R8: renamed from R17; value 330R -> 330; footprint Resistors_SMD:R_0805_HandSoldering -> Resistor_SMD:R_0805_2012Metric; symbol R_Small -> Device:R_Small
- R9: renamed from R21; value 330R -> 330; footprint Resistors_SMD:R_0805_HandSoldering -> Resistor_SMD:R_0805_2012Metric; symbol R_Small -> Device:R_Small
- SW1: footprint Buttons_Switches_THT:SW_PUSH_6mm -> Button_Switch_THT:SW_PUSH_6mm; symbol SW_Push -> Switch:SW_Push
- TP1: renamed from TP26; footprint Measurement_Points:Test_Point_Keystone_5005-5009_Compact -> TestPoint:TestPoint_Keystone_5005-5009_Compact; symbol TEST -> Connector:TestPoint
- TP10: renamed from TP3; footprint Measurement_Points:Test_Point_Keystone_5005-5009_Compact -> TestPoint:TestPoint_Keystone_5005-5009_Compact; symbol TEST -> Connector:TestPoint
- TP11: renamed from TP23; footprint Measurement_Points:Test_Point_Keystone_5005-5009_Compact -> TestPoint:TestPoint_Keystone_5005-5009_Compact; symbol TEST -> Connector:TestPoint
- TP12: renamed from TP2; footprint Measurement_Points:Test_Point_Keystone_5005-5009_Compact -> TestPoint:TestPoint_Keystone_5005-5009_Compact; symbol TEST -> Connector:TestPoint
- TP13: renamed from TP12; footprint Measurement_Points:Test_Point_Keystone_5005-5009_Compact -> TestPoint:TestPoint_Keystone_5005-5009_Compact; symbol TEST -> Connector:TestPoint
- TP14: renamed from TP4; footprint Measurement_Points:Test_Point_Keystone_5005-5009_Compact -> TestPoint:TestPoint_Keystone_5005-5009_Compact; symbol TEST -> Connector:TestPoint
- TP15: renamed from TP25; footprint Measurement_Points:Test_Point_Keystone_5005-5009_Compact -> TestPoint:TestPoint_Keystone_5005-5009_Compact; symbol TEST -> Connector:TestPoint
- TP16: renamed from TP24; footprint Measurement_Points:Test_Point_Keystone_5005-5009_Compact -> TestPoint:TestPoint_Keystone_5005-5009_Compact; symbol TEST -> Connector:TestPoint
- TP17: renamed from TP9; footprint Measurement_Points:Test_Point_Keystone_5005-5009_Compact -> TestPoint:TestPoint_Keystone_5005-5009_Compact; symbol TEST -> Connector:TestPoint
- TP18: renamed from TP10; footprint Measurement_Points:Test_Point_Keystone_5005-5009_Compact -> TestPoint:TestPoint_Keystone_5005-5009_Compact; symbol TEST -> Connector:TestPoint
- TP19: renamed from TP7; footprint Measurement_Points:Test_Point_Keystone_5005-5009_Compact -> TestPoint:TestPoint_Keystone_5005-5009_Compact; symbol TEST -> Connector:TestPoint
- TP2: renamed from TP11; footprint Measurement_Points:Test_Point_Keystone_5005-5009_Compact -> TestPoint:TestPoint_Keystone_5005-5009_Compact; symbol TEST -> Connector:TestPoint
- TP20: renamed from TP8; footprint Measurement_Points:Test_Point_Keystone_5005-5009_Compact -> TestPoint:TestPoint_Keystone_5005-5009_Compact; symbol TEST -> Connector:TestPoint
- TP21: renamed from TP19; footprint Measurement_Points:Test_Point_Keystone_5005-5009_Compact -> TestPoint:TestPoint_Keystone_5005-5009_Compact; symbol TEST -> Connector:TestPoint
- TP22: renamed from TP20; footprint Measurement_Points:Test_Point_Keystone_5005-5009_Compact -> TestPoint:TestPoint_Keystone_5005-5009_Compact; symbol TEST -> Connector:TestPoint
- TP23: renamed from TP13; footprint Measurement_Points:Test_Point_Keystone_5005-5009_Compact -> TestPoint:TestPoint_Keystone_5005-5009_Compact; symbol TEST -> Connector:TestPoint
- TP24: renamed from TP14; footprint Measurement_Points:Test_Point_Keystone_5005-5009_Compact -> TestPoint:TestPoint_Keystone_5005-5009_Compact; symbol TEST -> Connector:TestPoint
- TP25: renamed from TP15; footprint Measurement_Points:Test_Point_Keystone_5005-5009_Compact -> TestPoint:TestPoint_Keystone_5005-5009_Compact; symbol TEST -> Connector:TestPoint
- TP26: renamed from TP16; footprint Measurement_Points:Test_Point_Keystone_5005-5009_Compact -> TestPoint:TestPoint_Keystone_5005-5009_Compact; symbol TEST -> Connector:TestPoint
- TP27: renamed from TP21; footprint Measurement_Points:Test_Point_Keystone_5005-5009_Compact -> TestPoint:TestPoint_Keystone_5005-5009_Compact; symbol TEST -> Connector:TestPoint
- TP28: renamed from TP22; footprint Measurement_Points:Test_Point_Keystone_5005-5009_Compact -> TestPoint:TestPoint_Keystone_5005-5009_Compact; symbol TEST -> Connector:TestPoint
- TP3: renamed from TP27; footprint Measurement_Points:Test_Point_Keystone_5005-5009_Compact -> TestPoint:TestPoint_Keystone_5005-5009_Compact; symbol TEST -> Connector:TestPoint
- TP4: renamed from TP28; footprint Measurement_Points:Test_Point_Keystone_5005-5009_Compact -> TestPoint:TestPoint_Keystone_5005-5009_Compact; symbol TEST -> Connector:TestPoint
- TP5: renamed from TP17; footprint Measurement_Points:Test_Point_Keystone_5005-5009_Compact -> TestPoint:TestPoint_Keystone_5005-5009_Compact; symbol TEST -> Connector:TestPoint
- TP6: renamed from TP18; footprint Measurement_Points:Test_Point_Keystone_5005-5009_Compact -> TestPoint:TestPoint_Keystone_5005-5009_Compact; symbol TEST -> Connector:TestPoint
- TP7: renamed from TP5; footprint Measurement_Points:Test_Point_Keystone_5005-5009_Compact -> TestPoint:TestPoint_Keystone_5005-5009_Compact; symbol TEST -> Connector:TestPoint
- TP8: renamed from TP6; value GNDP -> Device GND; footprint Measurement_Points:Test_Point_Keystone_5005-5009_Compact -> TestPoint:TestPoint_Keystone_5005-5009_Compact; symbol TEST -> Connector:TestPoint
- TP9: renamed from TP1; footprint Measurement_Points:Test_Point_Keystone_5005-5009_Compact -> TestPoint:TestPoint_Keystone_5005-5009_Compact; symbol TEST -> Connector:TestPoint
- U1: renamed from U2; footprint UTSVT_Special:NucleoL432KC -> MPPT-PrimaryPCB:MODULE_NUCLEO-L432KC; symbol Nucleo_L432KC -> Array:MCU_Nucleo_L432KC
- U2: renamed from U3; footprint UTSVT_ICs:SOIC-8_4.00x5.00mm_Pitch1.27mm -> Package_SO:SOIC-8_3.9x4.9mm_P1.27mm; symbol UCC37321 -> Array:UCC37321
- U3: renamed from U1; footprint UTSVT_ICs:CUI_PQMC3-S -> MPPT-PrimaryPCB:490_PQMC3_D12_S12_S; symbol PQMC3-Dx-Sx-S -> Array:PWR_REG_PQMC3-Dx-Sx-S
- U4: footprint UTSVT_ICs:SOIC-6_1.40x2.15mm_Pitch0.65mm -> MPPT-PrimaryPCB:SC70-6; symbol INA21x -> Array:OP_AMP_INA21x
- U5: renamed from U6; footprint UTSVT_ICs:SOIC-6_1.40x2.15mm_Pitch0.65mm -> MPPT-PrimaryPCB:SC70-6; symbol INA21x -> Array:OP_AMP_INA21x
- U8: renamed from U5; footprint UTSVT_ICs:SOIC-20W_7.5x15.4mm_Pitch1.27mm -> MPPT-PrimaryPCB:ADM3055EBRIZ; symbol ADM3055E -> Array:CAN_Chip_ADM3055E
- U9: renamed from U7; footprint TO_SOT_Packages_SMD:SOT-23W_Handsoldering -> Package_TO_SOT_SMD:SOT-23; symbol CDSOT23-T24CAN -> Array:CAN_Bus_Protector_CDSOT23-T24CAN
Connections:
- net +3V3: now also U6.6 (VDD), U7.6 (VDD)
- net +Arr: now also F1.2; no longer J2.1 (+)
- net -Arr: now also J2.2 (-); no longer J2.3 (-)
- net Array_Current: now also U1.24 (A5); no longer U1.22 (A3)
- net Array_Voltage: now also U1.25 (A6), U6.1, U6.4 (IN-); no longer C15.1, R20.2, U1.24 (A5)
- net Battery_Current: now also U1.22 (A3); no longer U1.21 (A2)
- net Battery_Voltage: now also U7.1, U7.4 (IN-); no longer C16.1, R23.2
- net GNDPWR: now also C4.2, C5.2, J1.2 (GND), LED3.1 (K), TP6.1, U3.1 (GND); no longer C1.1, C10.2, C11.2, C12.2, C13.2, C14.2, C15.2, C16.2, C17.2, C18.2, C19.2, C2.2, C20.2, C3.2, C6.1, C7.2, C8.2, C9.2, D1.2 (A), D10.2 (A), D11.2 (A), D12.2 (A), D13.2 (A), D14.2 (A), D2.2 (A), D3.2 (A), D7.2 (A), D8.2 (A), D9.2 (A), LED4.1 (K), LED6.1 (K), LED7.1 (K), LED8.1 (K), LED9.1 (K), Q1.3 (S), Q2.3 (S), R12.2, R14.1, R16.2, R19.2, R22.2, SW1.1, TP1.1, TP15.1, TP3.1, TP4.1, TP8.1, U1.29 (GND), U1.4 (GND), U2.4 (AGND), U2.5 (PGND), U3.7 (0V), U4.1 (REF), U4.2 (V-), U4.4 (+), U5.1 (REF), U5.2 (V-), U5.5 (-), U8.1 (GND_In), U8.10 (GND_In), U8.2 (GND_In)
- net GNDREF: now also C1.1, C10.2, C11.2, C12.2, C13.2, C14.2, C15.2, C16.2, C17.2, C18.2, C19.2, C2.2, C20.2, C3.2, C6.1, C7.2, C8.2, C9.2, D1.2 (A), D10.2 (A), D11.2 (A), D12.2 (A), D13.2 (A), D14.2 (A), D2.2 (A), D3.2 (A), D7.2 (A), D8.2 (A), D9.2 (A), LED4.1 (K), LED6.1 (K), LED7.1 (K), LED8.1 (K), LED9.1 (K), Q1.3 (S), Q2.3 (S), R12.2, R14.1, R16.2, R19.2, R22.2, SW1.2, TP1.1, TP15.1, TP3.1, TP4.1, TP8.1, U1.29 (GND), U1.4 (GND), U2.4 (AGND), U2.5 (PGND), U3.7 (0V), U4.1 (REF), U4.2 (V-), U4.4 (+), U5.1 (REF), U5.2 (V-), U5.5 (-), U8.1 (GND_In), U8.10 (GND_In), U8.2 (GND_In), LED10.1 (K), LED5.1 (K), SW2.1, SW2.2, U6.2 (VSS), U7.2 (VSS); no longer C4.2, C5.2, J1.2 (GND), LED3.1 (K), TP6.1, U3.1 (GND)
- net Reset: now also SW1.1; no longer SW1.2
- net at U1.10 (D7): now also SW2.4
- net at U1.11 (D8): now also SW2.3
- net BPS_Full: now reaches U1.12 (D9)
- net BPS_Full: now also R11.2
- net at C23.1, C24.1, J4.1 (5V)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: now also C22.1; no longer C21.1
- net at C23.2, C24.2, J4.2 (GND)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: now also C22.2; no longer C21.2
- net at L3.2, TP23.1, U8.19 (V_ISO_Out): now also C21.1; no longer C22.1
- net at L4.2, TP26.1, U8.18 (GND_ISO_Out)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: now also C21.2; no longer C22.2
- net Battery_Full renamed Error
- net Error: now also R6.2
- new net: F1.1, J2.1 (+)
- new net: C15.1, R20.2, U6.3 (IN+)
- new net: C16.1, R23.2, U7.3 (IN+)
- new net: LED10.2 (A), R11.1
- new net: LED5.2 (A), R6.1
- no-connect marks 15 -> 18
Other:
- note added: "Changes from 3.1+:\n\nSchematic:\n- Reannotated all component labels and reverted rescued schematic symbols.\n- Rearranged schematic and cleaned up component positioning.\n- Created Array.lib for array-relevant schematic symbols.\n- Swapped out zener diodes going into the uC from 3.6V to 3.9V.\n- Updated the LEDs and resistors for Xx_live indicators.\n- Added Error indicator LED.\n- Shifted pins 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"
- note added: "For decoupling, we\nadd extra capacitors\nand unlink the power\npins on either side."
- note added: "Isolated Power Regions:\n* Device/Board Power\n - +/-Arr\n - +/-Batt\n - +9VA, +5V, +3.3V\n - GNDREF\n* Car Power\n - +12V\n - GNDPWR"
- note added: "Note that A7 (PA2) and A2 (PA3) are reserved \nfor STLink UART."
- note added: "R13, C9 are experimental and are through \nhole components with a range of values."
- note added: "USB"
- note removed: "Basic voltage\ndividers"
- note removed: "For decoupling, we\nadd extra capacitors\nand unlink the power\npins on either side"
- note removed: "Isolated Power Regions:\n* High Power/Nucleo\n - +/-Arr\n - +/-Batt\n - +9A, +5V, +3.3V\n - GNDPWR\n* Low Car Power\n - +12V\n - GNDREF"
- note removed: "RC filter\noptional"
- note removed: "filter\noptional"
- note removed: "pi filter\noptional"
- moved on the sheet: C1, C10, C11, C12, C13, C14, C15, C16, C17, C18, C19, C2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
